File: dioBreakOutBoard 1/dioBreakOutBoard/dioBreakOutBoard.kicad_pcb (KiCad board)
At the start: 4 copper layers, 116.2 x 190.5 mm, 75 parts, among them IC1 24AA025E48-E_SN, J1 Conn_01x03_Pin, J11 56509455, J12 56509455, J2 Samtec_ASP-134602-01, P1 Samtec_ASP-134606-01, U1 SN74LVC8T245QPWRQ1, U2 SN74LVC8T245QPWRQ1, U3 SN74LVC8T245QPWRQ1, U4 SN74LVC8T245QPWRQ1, U5 SN74LVC8T245QPWRQ1, U6 SN74LVC8T245QPWRQ1, U7 SN74LVC8T245QPWRQ1, U8 SN74LVC8T245QPWRQ1

Commit message: More routing done
Connections:
- U6 pad 10: FMC0_LA23.N -> FMC0_LA23.P
- U6 pad 5: FMC0_LA21.P -> FMC0_LA21.N
- U6 pad 6: FMC0_LA21.N -> FMC0_LA21.P
- U6 pad 7: FMC0_LA22.P -> FMC0_LA22.N
- U6 pad 8: FMC0_LA22.N -> FMC0_LA22.P
- U6 pad 9: FMC0_LA23.P -> FMC0_LA23.N
Routing:
- net FMC0_LA05.N: track 0.00 -> 106.8 mm, vias 1 -> 2
- net FMC0_LA07.N: track 0.00 -> 102.5 mm, vias 1 -> 2
- net FMC0_LA07.P: track 0.00 -> 101.0 mm, vias 1 -> 2
- net FMC0_LA06.N: track 0.00 -> 98.8 mm
- net FMC0_LA06.P: track 0.00 -> 95.7 mm
- net FMC0_LA05.P: track 0.00 -> 94.8 mm
- net FMC0_LA04.N: track 0.00 -> 92.2 mm, vias 1 -> 2
- net FMC0_LA04.P: track 0.00 -> 90.3 mm
- net FMC0_LA11.N: track 0.00 -> 83.8 mm, vias 1 -> 2
- net FMC0_LA11.P: track 0.00 -> 82.8 mm, vias 1 -> 2
- net FMC0_LA10.N: track 0.00 -> 82.6 mm, vias 1 -> 2
- net FMC0_LA09.N: track 0.00 -> 81.1 mm, vias 1 -> 2
- net FMC0_LA10.P: track 0.00 -> 80.8 mm, vias 1 -> 2
- net FMC0_LA09.P: track 0.00 -> 78.5 mm, vias 1 -> 2
- net FMC0_LA08.N: track 0.00 -> 77.1 mm, vias 1 -> 2
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