File: dioBreakOutBoard 1/dioBreakOutBoard/p1_fmc_connector.kicad_sch (KiCad schematic)
At the start: 9 parts, among them IC1 24AA025E48-E_SN, J2 Samtec_ASP-134602-01

Commit message: C:\Users\khernandez\KiCad\KiCad-Projects# Please enter the commit message for your changes. Lines starting
Parts:
- added C10, C8: 1u, Capacitor_SMD:C_0805_2012Metric_Pad1.18x1.45mm_HandSolder, symbol Device:C
- added C3, C9: 4.7u, Capacitor_SMD:C_1206_3216Metric, symbol Device:C
Connections:
- net FMC0_DP0.P is gone; now on net GND: J2.C2 (Pin_2), J2.C6 (Pin_6)
- net FMC0_DP1.N is gone; now on net +1V8: J2.A23 (Pin_23), J2.A3 (Pin_3)
- net FMC0_DP1.P is gone; now on net GND: J2.A2 (Pin_2), J2.A22 (Pin_22)
- net FMC0_DP2.N is gone; now on net +1V8: J2.A27 (Pin_27), J2.A7 (Pin_7)
- net FMC0_DP2.P is gone; now on net GND: J2.A26 (Pin_26), J2.A6 (Pin_6)
- net FMC0_DP3.N is gone; now on net +1V8: J2.A11 (Pin_11), J2.A31 (Pin_31)
- net FMC0_DP3.P is gone; now on net GND: J2.A10 (Pin_10), J2.A30 (Pin_30)
- net +1V8: now also J2.C7 (Pin_7), C10.2, C9.2
- net +3V3: now also J2.D32 (Pin_32), C3.2, C8.2
- net GND: now also J2.C3 (Pin_3), C10.1, C3.1, C8.1, C9.1
- net HA01_CC.P: now reaches J2.E2 (Pin_2)
- net HA01_CC.N: now reaches J2.E3 (Pin_3)
- net +3.3VA renamed +3.3V
- net +3.3V: no longer J2.D32 (Pin_32)
- removed net FMC0_DP0.N: J2.C3 (Pin_3), J2.C7 (Pin_7)
- net FMC0_HA05.N renamed HA05.N
- net FMC0_HA05.P renamed HA05.P
- no-connect marks 120 -> 134
Other:
- note removed: "GBT LOOP BACKS"

Commit message: added 2 bit buffers, which replace the previous 8 bit buffers
Parts:
- renumbered C9 to C1, C3 to C2, C10 to C3, C8 to C4, C1 to C5, C2 to C6, J2 to J1, R4 to R1, R5 to R2, TP4 to TP1, TP1 to TP3
